File: hardware/kicad/z80_romless_sbc.kicad_sch (KiCad schematic)
At the start: 56 parts, among them J1 REGULATED 5V INPUT, U1 Z84C0020PEC, U2 AS6C1008-55PCN, U3 ATF22V10B/C, U4 SN74HCT541N, U5 SN74HCT245N LOW, U6 SN74HCT245N HIGH, U7 SN74LVC244AN, U8 MCP23S17-E/SP, U9 SN74LVC8T245PW

Commit message: Refactor bus control and update schematic definitions
- Updated pin definitions in bus.h and pins.h to replace unused pins with DATA_ENABLE and ADDR_ENABLE.
- Refactored bus.c to remove the z80_set_transceiver function and replace its calls with direct GPIO manipulations for address and data bus control.
- Modified build-kicad-schematic.py to reflect new pin names and added new components (NPN transistor and resistors) for MCP reset functionality.
- Adjusted the README.md files to clarify testing procedures and updated stage descriptions in main.c files for various stages.
- Enhanced PDF generation in build-readme-pdf.mjs to include page numbers in the footer.
Parts:
- removed C13: 10u Peripheral Board, Capacitor_THT:C_Disc_D5.0mm_W2.5mm_P2.50mm, symbol Z80SBC:CAPACITOR
- removed C14: 47u Supply Entry, Capacitor_THT:C_Disc_D5.0mm_W2.5mm_P2.50mm, symbol Z80SBC:CAPACITOR
- removed U5: SN74HCT245N LOW, Package_DIP:DIP-20_W7.62mm, symbol Z80SBC:HCT245
- removed U6: SN74HCT245N HIGH, Package_DIP:DIP-20_W7.62mm, symbol Z80SBC:HCT245
- added Q1: 2N3904 MCP RESET, Package_TO_SOT_THT:TO-92_Inline, symbol Z80SBC:NPN
- added R30: 47k MCP reset base pull-down, Resistor_THT:R_Axial_DIN0207_L6.3mm_D2.5mm_P10.16mm_Horizontal, symbol Z80SBC:RESISTOR
- added R31: 10k MCP RESET# pull-up, Resistor_THT:R_Axial_DIN0207_L6.3mm_D2.5mm_P10.16mm_Horizontal, symbol Z80SBC:RESISTOR
- added RN1: 8x10k A0-A7 pull-up, symbol Z80SBC:RN8
- added RN2: 8x10k A8-A15 pull-up, symbol Z80SBC:RN8
- added RN3: 8x10k Pico D0-D7 pull-down, symbol Z80SBC:RN8
- added U10: SN74LVC245AN bus-to-Pico, Package_DIP:DIP-20_W7.62mm, symbol Z80SBC:LVC245
- C10: value 100n U9 VCCB -> 22u Core Board
- C11: value 10u Memory Board -> 22u Peripheral Board
- C12: value 10u Core Board -> 100u Supply Entry
- C5: value 100n U5 HCT245 -> 100n U7 LVC244
- C6: value 100n U6 HCT245 -> 100n U8 MCP
- C7: value 100n U7 LVC244 -> 100n U9 AHCT245
- C8: value 100n U8 MCP -> 100n U10 LVC245
- C9: value 100n U9 VCCA -> 22u Memory Board
- R19: value 10k DATA_OE_N -> 10k PICO_SPI_CS_N
- R20: value 10k ADDR_OE_N -> 10k PICO_WE_N
- R21: value 10k PICO_SPI_CS_N -> 10k PICO_OE_N
- R22: value 10k PICO_WE_N -> 10k PICO_CLK
- R23: value 10k PICO_OE_N -> 10k RESET_N
- R24: value 10k PICO_CLK -> 10k DATA_ENABLE
- R25: value 10k RESET_N -> 10k DATA_DIR
- R26: value 10k DATA_DIR -> 10k ADDR_ENABLE
- R27: value 10k ADDR_DIR -> 10k PICO_SPI_SCK
- R28: value 10k PICO_SPI_SCK -> 10k PICO_SPI_MOSI
- R29: value 10k PICO_SPI_MOSI -> 4.7k MCP reset base
- U9: value SN74LVC8T245PW -> SN74AHCT245N Pico-to-bus; footprint Package_DIP:DIP-24_W15.24mm -> Package_DIP:DIP-20_W7.62mm; symbol Z80SBC:LVC8T245 -> Z80SBC:AHCT245
Connections:
- net MCP_GPA0 is gone; now on net A0: U8.21 (GPA0)
- net MCP_GPA1 is gone; now on net A1: U8.22 (GPA1)
- net MCP_GPA2 is gone; now on net A2: U8.23 (GPA2)
- net MCP_GPA3 is gone; now on net A3: U8.24 (GPA3)
- net MCP_GPA4 is gone; now on net A4: U8.25 (GPA4)
- net MCP_GPA5 is gone; now on net A5: U8.26 (GPA5)
- net MCP_GPA6 is gone; now on net A6: U8.27 (GPA6)
- net MCP_GPA7 is gone; now on net A7: U8.28 (GPA7)
- net MCP_GPB0 is gone; now on net A8: U8.1 (GPB0)
- net MCP_GPB1 is gone; now on net A9: U8.2 (GPB1)
- net MCP_GPB2 is gone; now on net A10: U8.3 (GPB2)
- net MCP_GPB3 is gone; now on net A11: U8.4 (GPB3)
- net MCP_GPB4 is gone; now on net A12: U8.5 (GPB4)
- net MCP_GPB5 is gone; now on net A13: U8.6 (GPB5)
- net MCP_GPB6 is gone; now on net A14: U8.7 (GPB6)
- net MCP_GPB7 is gone; now on net A15: U8.8 (GPB7)
- net +3V3: now also C5.1 (+), C8.1 (+), U10.20 (VCC); no longer C7.1 (+), C9.1 (+), R22.2, R23.2, U9.1 (VCCA)
- net +5V: now also C7.1 (+), C9.1 (+), U9.1 (DIR), U9.20 (VCC), R31.2, RN1.1 (COMMON), RN2.1 (COMMON); no longer C5.1 (+), C8.1 (+), U8.18 (RESET#), U9.23 (VCCB1), U9.24 (VCCB2)
- net A0: now also RN1.2 (R1)
- net A1: now also RN1.3 (R2)
- net A10: now also RN2.4 (R3)
- net A11: now also RN2.5 (R4)
- net A12: now also RN2.6 (R5)
- net A13: now also RN2.7 (R6)
- net A14: now also RN2.8 (R7)
- net A15: now also RN2.9 (R8)
- net A2: now also RN1.4 (R3)
- net A3: now also RN1.5 (R4)
- net A4: now also RN1.6 (R5)
- net A5: now also RN1.7 (R6)
- net A6: now also RN1.8 (R7)
- net A7: now also RN1.9 (R8)
- net A8: now also RN2.2 (R1)
- net A9: now also RN2.3 (R2)
- net D0: now also U9.18 (B1), U10.18 (B1); no longer U9.21 (B1)
- net D1: now also U9.17 (B2), U10.17 (B2); no longer U9.20 (B2)
- net D2: now also U9.16 (B3), U10.16 (B3); no longer U9.19 (B3)
- net D3: now also U9.15 (B4), U10.15 (B4); no longer U9.18 (B4)
- net D4: now also U9.14 (B5), U10.14 (B5); no longer U9.17 (B5)
- net D5: now also U9.13 (B6), U10.13 (B6); no longer U9.16 (B6)
- net D6: now also U9.12 (B7), U10.12 (B7); no longer U9.15 (B7)
- net D7: now also U9.11 (B8), U10.11 (B8); no longer U9.14 (B8)
- net DATA_DIR: now also R25.1, U3.11 (DATA_DIR); no longer R26.1, U9.2 (DIR)
- net GND: now also R22.2, R23.2, U9.10 (GND), Q1.1 (E), R30.2, RN3.1 (COMMON), U10.1 (DIR), U10.10 (GND); no longer R29.2, U3.10 (UNUSED_IN2), U3.11 (UNUSED_IN3), U3.9 (UNUSED_IN1), U9.11 (GND1), U9.12 (GND2), U9.13 (GND3)
- net PICO_CLK: now also R22.1; no longer R24.1
- net PICO_D0: now also U9.2 (A1), RN3.2 (R1), U10.2 (A1); no longer U9.3 (A1)
- net PICO_D1: now also U9.3 (A2), RN3.3 (R2), U10.3 (A2); no longer U9.4 (A2)
- net PICO_D2: now also U9.4 (A3), RN3.4 (R3), U10.4 (A3); no longer U9.5 (A3)
- net PICO_D3: now also U9.5 (A4), RN3.5 (R4), U10.5 (A4); no longer U9.6 (A4)
- net PICO_D4: now also U9.6 (A5), RN3.6 (R5), U10.6 (A5); no longer U9.7 (A5)
- net PICO_D5: now also U9.7 (A6), RN3.7 (R6), U10.7 (A6); no longer U9.8 (A6)
- net PICO_D6: now also U9.8 (A7), RN3.8 (R7), U10.8 (A7); no longer U9.9 (A7)
- net PICO_D7: now also U9.9 (A8), RN3.9 (R8), U10.9 (A8); no longer U9.10 (A8)
- net PICO_OE_N: now also R21.1; no longer R23.1
- net PICO_SPI_CS_N: now also R19.1; no longer R21.1
- net PICO_SPI_MOSI: now also R28.1; no longer R29.1
- net PICO_SPI_SCK: now also R27.1; no longer R28.1
- net PICO_WE_N: now also R20.1; no longer R22.1
- net RESET_N: now also R23.1; no longer R25.1
- net DATA_UP_OE_N: now reaches U3.17 (DATA_UP_OE#)
- net DATA_UP_OE_N: now also U9.19 (OE#)
- net DATA_DOWN_OE_N: now reaches U3.18 (DATA_DOWN_OE#)
- net DATA_DOWN_OE_N: now also U10.19 (OE#)
- net MCP_RESET_DRIVE: now reaches U3.19 (MCP_RESET_DRIVE)
- net MCP_RESET_DRIVE: now also R29.1
- net ADDR_DIR: no longer names the net of A1.11 (GP8)
- net ADDR_DIR: no longer R27.1
- net ADDR_OE_N renamed ADDR_ENABLE
- net ADDR_ENABLE: now also R26.1, U3.10 (ADDR_ENABLE); no longer R20.1
- removed net DATA_OE_N: A1.10 (GP7), R19.1, U9.22 (OE#)
- new net DATA_ENABLE: A1.10 (GP7), R24.1, U3.9 (DATA_ENABLE)
- new net MCP_RESET_BASE: Q1.2 (B), R29.2, R30.1
- new net MCP_RESET_N: Q1.3 (C), R31.1, U8.18 (RESET#)
- no-connect marks 19 -> 17
Other:
- note added: "ADDRESS_RESET"
- note added: "R1-R16: 5V fail-safe pulls. R17-R21: 3V3 pulls. R22-R28: GPIO pull-downs. R29-R31: MCP reset transistor bias."
- note removed: "ADDRESS_CONTROL"
- note removed: "MCP_GPA"
- note removed: "MCP_GPB"
- note removed: "Startup pulls: R1-R16 = 5V pull-ups, R17-R23 = 3V3 pull-ups, R24-R29 = 3V3-side pull-downs."
- moved on the sheet: R29, U8

Commit message: Refactor breadboard layout and schematic to replace SN74HCT541N with SN74AHCT244N
- Updated breadboard layout SVG to reflect the change from HCT541 to AHCT244.
- Modified build-breadboard-layout script to replace references to HCT541 with AHCT244.
- Adjusted KiCad schematic generation script to update component details and pin assignments for AHCT244.
- Increased maximum clock frequency in clock.c from 4MHz to 8MHz.
- Enhanced IO trap handling in io_trap.c for better control flow and timeout management.
- Updated SRAM control PLD to reflect changes in pin assignments and added WAIT_N logic.
- Changed main.c output message to indicate the use of AHCT244 instead of HCT541.
Parts:
- C4: value 100n U4 HCT541 -> 100n U4 AHCT244
- U4: value SN74HCT541N -> SN74AHCT244N; symbol Z80SBC:HCT541 -> Z80SBC:AHCT244
Connections:
- net BUSREQ_N: now also U4.16 (1Y2); no longer U4.17 (Y2)
- net GND: no longer U3.13 (UNUSED_IN4)
- net IORQ_N: now also U3.13 (Z80_IORQ#)
- net MCP_CS_N: now also U4.14 (1Y3); no longer U4.16 (Y3)
- net MCP_SCK: now also U4.12 (1Y4); no longer U4.15 (Y4)
- net MCP_SI: now also U4.9 (2Y1); no longer U4.14 (Y5)
- net PICO_BUSREQ_N: now also U4.4 (1A2); no longer U4.3 (A2)
- net PICO_SPI_CS_N: now also U4.6 (1A3); no longer U4.4 (A3)
- net PICO_SPI_MOSI: now also U4.11 (2A1); no longer U4.6 (A5)
- net PICO_SPI_SCK: now also U4.8 (1A4); no longer U4.5 (A4)
- net SRAM_CE_N: now also U4.3 (2Y4); no longer U4.11 (Y8)
- net SRAM_CE_PRE_N: now also U4.17 (2A4); no longer U4.9 (A8)
- net SRAM_OE_N: now also U4.5 (2Y3); no longer U4.12 (Y7)
- net SRAM_OE_PRE_N: now also U4.15 (2A3); no longer U4.8 (A7)
- net SRAM_WE_N: now also U4.7 (2Y2); no longer U4.13 (Y6)
- net SRAM_WE_PRE_N: now also U4.13 (2A2); no longer U4.7 (A6)
- net WAIT_N: now also U3.20 (WAIT#)
- no-connect marks 17 -> 16
