File: hardware/kicad/z80_romless_sbc.kicad_sch (KiCad schematic)
At the start: 59 parts, among them J1 REGULATED 5V INPUT, Q1 2N3904 MCP RESET, U1 Z84C0020PEC, U10 SN74LVC245AN bus-to-Pico, U2 AS6C1008-55PCN, U3 ATF22V10B/C, U4 SN74AHCT244N, U7 SN74LVC244AN, U8 MCP23S17-E/SP, U9 SN74AHCT245N Pico-to-bus

Commit message: Enhance KiCad schematic and build scripts
- Updated `build-kicad-schematic.py` to include component descriptions in properties and added a new dictionary to store component details.
- Refactored component addition calls to include descriptions for resistors and capacitors.
- Improved the handling of temporary directories in `build-kicad.sh` for better organization of generated files.
- Added checks for KiCad Python environment and improved error handling for missing routing sessions.
- Enhanced export commands in the build script to include additional formats and organized output into structured directories.
Parts:
- added TP2: CLK TEST, TestPoint:TestPoint_Loop_D2.60mm_Drill0.9mm_Beaded, symbol Z80SBC:TESTPOINT
- added TP3: RESET# TEST, TestPoint:TestPoint_Loop_D2.60mm_Drill0.9mm_Beaded, symbol Z80SBC:TESTPOINT
- added TP4: WAIT# TEST, TestPoint:TestPoint_Loop_D2.60mm_Drill0.9mm_Beaded, symbol Z80SBC:TESTPOINT
- added TP5: BUSREQ# TEST, TestPoint:TestPoint_Loop_D2.60mm_Drill0.9mm_Beaded, symbol Z80SBC:TESTPOINT
- added TP6: BUSACK# TEST, TestPoint:TestPoint_Loop_D2.60mm_Drill0.9mm_Beaded, symbol Z80SBC:TESTPOINT
- added TP7: GND TEST, TestPoint:TestPoint_Loop_D2.60mm_Drill0.9mm_Beaded, symbol Z80SBC:TESTPOINT
- C1: value 100n U1 Z80 -> 100n
- C10: value 22u Core Board -> 22u; footprint Capacitor_THT:C_Disc_D5.0mm_W2.5mm_P2.50mm -> Capacitor_THT:CP_Radial_D8.0mm_P3.50mm
- C11: value 22u Peripheral Board -> 22u; footprint Capacitor_THT:C_Disc_D5.0mm_W2.5mm_P2.50mm -> Capacitor_THT:CP_Radial_D8.0mm_P3.50mm
- C12: value 100u Supply Entry -> 100u; footprint Capacitor_THT:C_Disc_D5.0mm_W2.5mm_P2.50mm -> Capacitor_THT:CP_Radial_D10.0mm_P5.00mm
- C2: value 100n U2 SRAM -> 100n
- C3: value 100n U3 GAL -> 100n
- C4: value 100n U4 AHCT244 -> 100n
- C5: value 100n U7 LVC244 -> 100n
- C6: value 100n U8 MCP -> 100n
- C7: value 100n U9 AHCT245 -> 100n
- C8: value 100n U10 LVC245 -> 100n
- C9: value 22u Memory Board -> 22u; footprint Capacitor_THT:C_Disc_D5.0mm_W2.5mm_P2.50mm -> Capacitor_THT:CP_Radial_D8.0mm_P3.50mm
- J1: footprint (none) -> TerminalBlock_Altech:Altech_AK100_1x02_P5.00mm
- R1: value 10k BUSREQ_N -> 10k
- R10: value 10k SRAM_WE_N -> 10k
- R11: value 10k WAIT_N -> 10k
- R12: value 10k INT_N -> 10k
- R13: value 10k NMI_N -> 10k
- R14: value 10k SRAM_WE_PRE_N -> 10k
- R15: value 10k SRAM_OE_PRE_N -> 10k
- R16: value 10k SRAM_CE_PRE_N -> 10k
- R17: value 10k PICO_BUSREQ_N -> 10k
- R18: value 10k PICO_CE_N -> 10k
- R19: value 10k PICO_SPI_CS_N -> 10k
- R2: value 10k BUSACK_N -> 10k
- R20: value 10k PICO_WE_N -> 10k
- R21: value 10k PICO_OE_N -> 10k
- R22: value 10k PICO_CLK -> 10k
- R23: value 10k RESET_N -> 10k
- R24: value 10k DATA_ENABLE -> 10k
- R25: value 10k DATA_DIR -> 10k
- R26: value 10k ADDR_ENABLE -> 10k
- R27: value 10k PICO_SPI_SCK -> 10k
- R28: value 10k PICO_SPI_MOSI -> 10k
- R29: value 4.7k MCP reset base -> 4.7k
- R3: value 10k MREQ_N -> 10k
- R30: value 47k MCP reset base pull-down -> 47k
- R31: value 10k MCP RESET# pull-up -> 10k
- R4: value 10k IORQ_N -> 10k
- R5: value 10k RD_N -> 10k
- R6: value 10k WR_N -> 10k
- R7: value 10k MCP_SO -> 10k
- R8: value 10k SRAM_CE_N -> 10k
- R9: value 10k SRAM_OE_N -> 10k
- RN1: value 8x10k A0-A7 pull-up -> 8x10k bussed; footprint (none) -> Resistor_THT:R_Array_SIP9
- RN2: value 8x10k A8-A15 pull-up -> 8x10k bussed; footprint (none) -> Resistor_THT:R_Array_SIP9
- RN3: value 8x10k Pico D0-D7 pull-down -> 8x10k bussed; footprint (none) -> Resistor_THT:R_Array_SIP9
Connections:
- net BUSACK_N: now also TP6.1 (TP)
- net BUSREQ_N: now also TP5.1 (TP)
- net GND: now also TP7.1 (TP)
- net RESET_N: now also TP3.1 (TP)
- net WAIT_N: now also TP4.1 (TP)
- net Z80_CLK: now also TP2.1 (TP)
