File: hardware/kicad/z80_romless_sbc.kicad_sch (KiCad schematic)
At the start: 65 parts, among them J1 REGULATED 5V INPUT, Q1 2N3904 MCP RESET, U1 Z84C0020PEC, U10 SN74LVC245AN bus-to-Pico, U2 AS6C1008-55PCN, U3 ATF22V10B/C, U4 SN74AHCT244N, U7 SN74LVC244AN, U8 MCP23S17-E/SP, U9 SN74AHCT245N Pico-to-bus

Commit message: feat: consolidate control pull-ups
Replace sixteen discrete 10k control pull-ups with two functionally grouped bussed SIP networks, reroute the four-layer board, and regenerate validated documentation and fabrication outputs.

Co-authored-by: Copilot <223556219+Copilot@users.noreply.github.com>
Parts:
- removed R1, R10, R11, R12, R13, R14, R15, R16, R2, R3, R4, R5, R6, R7, R8, R9: 10k, Resistor_THT:R_Axial_DIN0207_L6.3mm_D2.5mm_P10.16mm_Horizontal, symbol Z80SBC:RESISTOR
- added RN4, RN5: 8x10k bussed, Resistor_THT:R_Array_SIP9, symbol Z80SBC:RN8
Connections:
- net +5V: now also RN4.1 (COMMON), RN5.1 (COMMON)
- net BUSACK_N: now also RN4.3 (R2)
- net BUSREQ_N: now also RN4.2 (R1)
- net INT_N: now also RN4.8 (R7)
- net IORQ_N: now also RN4.5 (R4)
- net MCP_SO: now also RN5.2 (R1)
- net MREQ_N: now also RN4.4 (R3)
- net NMI_N: now also RN4.9 (R8)
- net RD_N: now also RN4.6 (R5)
- net SRAM_CE_N: now also RN5.3 (R2)
- net SRAM_CE_PRE_N: now also RN5.9 (R8)
- net SRAM_OE_N: now also RN5.4 (R3)
- net SRAM_OE_PRE_N: now also RN5.8 (R7)
- net SRAM_WE_N: now also RN5.5 (R4)
- net SRAM_WE_PRE_N: now also RN5.7 (R6)
- net WAIT_N: now also RN5.6 (R5)
- net WR_N: now also RN4.7 (R6)
Other:
- note added: "RN4/RN5: 5V fail-safe pulls. R17-R21: 3V3 pulls. R22-R28: GPIO pull-downs. R29-R31: MCP reset transistor bias."
- note removed: "R1-R16: 5V fail-safe pulls. R17-R21: 3V3 pulls. R22-R28: GPIO pull-downs. R29-R31: MCP reset transistor bias."
- moved on the sheet: R17, R18, R19, R20, R21, R22, R23, R24, R25, R26, R27, R28
