File: hardware/kicad/z80_romless_sbc.kicad_sch (KiCad schematic)
At the start: 41 parts, among them J1 REGULATED 5V INPUT, J2 PICO GPIO EXPANSION, U1 Z84C0020PEC, U10 SN74LVC245AN bus-to-Pico, U2 AS6C1008-55PCN, U3 SN74HCT32N, U4 SN74AHCT244N, U7 SN74LVC244AN, U9 SN74AHCT245N Pico-to-bus

Commit message: - SRAM Memory Bank Switching Including:     - Updated BIOS     - Updated KiCad Schema - Remove Ctrl+s and print from CPM - Cleaned up docs - Z80 IO and IRQ Optimizations
Parts:
- added R24: 10k, Resistor_THT:R_Axial_DIN0207_L6.3mm_D2.5mm_P10.16mm_Horizontal, symbol Z80SBC:RESISTOR
Connections:
- net GND: now also R24.2; no longer U2.2 (A16), U4.17 (2A4)
- net PICO_GP8: now also U4.17 (2A4), R24.1
- net SRAM_A16: now reaches U4.3 (2Y4)
- net SRAM_A16: now also U2.2 (A16)
- no-connect marks 10 -> 9
Other:
- note added: "BANK SELECT: Pico physical pin 11 / GP8 -> U4.17. R24: 10k from Pico pin 11 to GND (3.3V side). U4.3 -> U2.2 / A16 (5V side); LOW selects bank 0. Remove the former U4.17 and U2.2 ground straps."
- note added: "J2: 3.3V signals only. Pin 1 / GP8 reserved for SRAM bank select. GP22/GP26 available for software/PIO I2C."
- note removed: "J2: 3.3V GPIO expansion only. No fixed pulls or level shifting. Use software/PIO for I2C or full-duplex SPI."
