File: hardware/kicad/z80_romless_sbc.kicad_pcb (KiCad board)
At the start: 4 copper layers, 160 x 135 mm, 55 parts, among them J1 REGULATED 5V INPUT, Q1 2N3904 MCP RESET, U1 Z84C0020PEC, U10 SN74LVC245AN bus-to-Pico, U2 AS6C1008-55PCN, U3 ATF22V10B/C, U4 SN74AHCT244N, U7 SN74LVC244AN, U8 MCP23S17-E/SP, U9 SN74AHCT245N Pico-to-bus

Commit message: Enhance PCB and schematic generation scripts, improve supervisor initialization, and expand test coverage
- Added +5V and GND assembly labels in build-kicad-pcb.py for better clarity.
- Updated build_board function to ensure correct layer settings for specific components.
- Implemented value checks for components in check_board function to ensure design integrity.
- Added checks for polarity silkscreen retention for capacitors C9 to C12.
- Modified resistor values in build-kicad-schematic.py based on signal requirements for improved circuit performance.
- Enhanced z80_safe_startup function in supervisor.c to initialize data pins correctly.
- Updated control_test to include supervisor.c for comprehensive testing.
- Expanded control_test.c with additional state tracking and assertions for safe startup and first write operations.
- Introduced sleep_ms function in fakes to simulate delays in tests.
- Included stdint.h in fakes/types.h for consistent type definitions.
Parts:
- R23, R24, R25, R26: value 10k -> 4.7k
Other:
- board text added: "+5V"
- board text added: "GND"
